Commit message: X7s code

File: X7S/meshes/X7S.urdf (robot description, URDF)
Before this commit: robot X7S, 23 links, 22 joints
Joints:
- joint joint10: limit lower=-3.141592653589793 upper=3.141592653589793 effort=100 velocity=1000 -> lower=-10 upper=10 effort=100 velocity=1000
- joint joint11: limit lower=-3.141592653589793 upper=3.141592653589793 effort=100 velocity=100 -> lower=-10 upper=10 effort=100 velocity=100
- joint joint14: limit lower=-3.141592653589793 upper=3.141592653589793 effort=100 velocity=1000 -> lower=-10 upper=10 effort=100 velocity=1000
- joint joint15: limit lower=-3.141592653589793 upper=3.141592653589793 effort=100 velocity=1000 -> lower=-10 upper=10 effort=100 velocity=1000
- joint joint16: limit lower=-3.141592653589793 upper=3.141592653589793 effort=100 velocity=1000 -> lower=-10 upper=10 effort=100 velocity=1000
- joint joint17: limit lower=-3.141592653589793 upper=3.141592653589793 effort=100 velocity=1000 -> lower=-10 upper=10 effort=100 velocity=1000
- joint joint18: limit lower=-3.141592653589793 upper=3.141592653589793 effort=100 velocity=1000 -> lower=-10 upper=10 effort=100 velocity=1000
- joint joint19: limit lower=-3.141592653589793 upper=3.141592653589793 effort=100 velocity=1000 -> lower=-10 upper=10 effort=100 velocity=1000
- joint joint2: limit lower=-1.57 upper=0.0 effort=100 velocity=1000 -> lower=-10 upper=10 effort=100 velocity=1000
- joint joint20: limit lower=-3.141592653589793 upper=3.141592653589793 effort=100 velocity=1000 -> lower=-10 upper=10 effort=100 velocity=1000
- joint joint3: limit lower=-3.141592653589793 upper=3.141592653589793 effort=100 velocity=1000 -> lower=-10 upper=10 effort=100 velocity=1000
- joint joint4: limit lower=-1.57 upper=1.57 effort=100 velocity=1000 -> lower=-10 upper=10 effort=100 velocity=1000
- joint joint5: limit lower=-3.141592653589793 upper=3.141592653589793 effort=100 velocity=1000 -> lower=-10 upper=10 effort=100 velocity=1000
- joint joint6: limit lower=-3.141592653589793 upper=3.141592653589793 effort=100 velocity=1000 -> lower=-10 upper=10 effort=100 velocity=1000
- joint joint7: limit lower=-3.141592653589793 upper=3.141592653589793 effort=100 velocity=1000 -> lower=-10 upper=10 effort=100 velocity=1000
- joint joint8: limit lower=-3.141592653589793 upper=3.141592653589793 effort=100 velocity=1000 -> lower=-10 upper=10 effort=100 velocity=1000
- joint joint9: limit lower=-3.141592653589793 upper=3.141592653589793 effort=100 velocity=1000 -> lower=-10 upper=10 effort=100 velocity=1000
